File: mk4-v1-board-with-fixes/kicad/fileOpamp1.sch (KiCad schematic (older format))
At the start: 7 parts, among them U2 LM358

Commit message: Soft push of v2 board modifications
Connections:
- net OUT1: now also R16.2, R18.2, U2.6 (-)
Changed lines of the file:
@@
 LIBS:valves
 LIBS:freetronics_schematic
+LIBS:cd4013b
 LIBS:hitchco-mk4-cache
 EELAYER 25 0
@@
 $Descr USLetter 11000 8500
 encoding utf-8
-Sheet 7 47
+Sheet 7 45
 Title "sensor-mcu"
 Date "2017-10-11"
@@
 $EndComp
 Wire Wire Line
-	5250 3850 5250 4250
+	5250 3850 5250 5050
 Wire Wire Line
 	4550 4250 4900 4250
@@
 	1    0    0    -1
 $EndComp
+Wire Wire Line
+	5250 5050 7150 5050
+Wire Wire Line
+	7150 5050 7150 4250
+Connection ~ 7150 4250
+Connection ~ 5250 4250
 $EndSCHEMATC
