File: mk4-v1-board-with-fixes/kicad/filePMOS1.sch (KiCad schematic (older format))
At the start: 7 parts, among them Q6 Q_PMOS_GDS, Q8 2N3904

Commit message: Soft push of v2 board modifications
Parts:
- R29, R31: value 1MΩ -> 10KΩ
Changed lines of the file:
@@
 LIBS:valves
 LIBS:freetronics_schematic
+LIBS:cd4013b
 LIBS:hitchco-mk4-cache
 EELAYER 25 0
@@
 $Descr USLetter 11000 8500
 encoding utf-8
-Sheet 20 47
+Sheet 18 45
 Title ""
 Date ""
@@
 AR Path="/59DEA30F/5A5D22C5/59E17AAC" Ref="Q25"  Part="1"
 AR Path="/59DEA30F/5A5D4870/59E17AAC" Ref="Q27"  Part="1"
-F 0 "Q15" H 4850 4875 50  0000 L CNN
+F 0 "Q13" H 4850 4875 50  0000 L CNN
 F 1 "2N3904" H 4850 4800 50  0000 L CNN
 F 2 "TO_SOT_Packages_THT:TO-92_Molded_Narrow" H 4850 4725 50  0001 L CIN
@@
 AR Path="/59DEA30F/5A5D22C5/59E17AB3" Ref="R81"  Part="1"
 AR Path="/59DEA30F/5A5D4870/59E17AB3" Ref="R85"  Part="1"
-F 0 "R45" V 4230 4800 50  0000 C CNN
+F 0 "R41" V 4230 4800 50  0000 C CNN
 F 1 "1KΩ" V 4150 4800 35  0000 C CNN
 F 2 "Resistors_THT:R_Axial_DIN0207_L6.3mm_D2.5mm_P10.16mm_Horizontal" V 4080 4800 50  0001 C CNN
@@
 AR Path="/59DEA30F/5A5D22C5/59E17ABB" Ref="R80"  Part="1"
 AR Path="/59DEA30F/5A5D4870/59E17ABB" Ref="R84"  Part="1"
-F 0 "R44" V 4830 4250 50  0000 C CNN
-F 1 "1MΩ" V 4750 4250 35  0000 C CNN
+F 0 "R40" V 4830 4250 50  0000 C CNN
+F 1 "10KΩ" V 4750 4250 35  0000 C CNN
 F 2 "Resistors_THT:R_Axial_DIN0207_L6.3mm_D2.5mm_P10.16mm_Horizontal" V 4680 4250 50  0001 C CNN
 F 3 "" H 4750 4250 50  0001 C CNN
@@
 AR Path="/59DEA30F/5A5D22C5/59E17AC2" Ref="R82"  Part="1"
 AR Path="/59DEA30F/5A5D4870/59E17AC2" Ref="R86"  Part="1"
-F 0 "R46" V 4430 5000 50  0000 C CNN
-F 1 "1MΩ" V 4350 5000 35  0000 C CNN
+F 0 "R42" V 4430 5000 50  0000 C CNN
+F 1 "10KΩ" V 4350 5000 35  0000 C CNN
 F 2 "Resistors_THT:R_Axial_DIN0207_L6.3mm_D2.5mm_P10.16mm_Horizontal" V 4280 5000 50  0001 C CNN
 F 3 "" H 4350 5000 50  0001 C CNN
@@
 AR Path="/59DEA30F/5A5D22C5/5A60FA4A" Ref="R83"  Part="1"
 AR Path="/59DEA30F/5A5D4870/5A60FA4A" Ref="R87"  Part="1"
-F 0 "R47" V 3880 5450 50  0000 C CNN
+F 0 "R43" V 3880 5450 50  0000 C CNN
 F 1 "330Ω" V 3800 5450 39  0000 C CNN
 F 2 "Resistors_THT:R_Axial_DIN0207_L6.3mm_D2.5mm_P10.16mm_Horizontal" V 3730 5450 50  0001 C CNN
@@
 AR Path="/59DEA30F/5A5D22C5/5A23876F" Ref="D14"  Part="1"
 AR Path="/59DEA30F/5A5D4870/5A23876F" Ref="D15"  Part="1"
-F 0 "D7" H 3800 5200 50  0000 C CNN
+F 0 "D6" H 3800 5200 50  0000 C CNN
 F 1 "LED" H 3800 5000 50  0000 C CNN
 F 2 "LEDs:LED_D5.0mm" H 3800 5100 50  0001 C CNN
@@
 AR Path="/59DEA30F/5A5D22C5/5A2F44DB" Ref="Q22"  Part="1"
 AR Path="/59DEA30F/5A5D4870/5A2F44DB" Ref="Q24"  Part="1"
-F 0 "Q12" H 5450 4550 50  0000 L CNN
+F 0 "Q11" H 5450 4550 50  0000 L CNN
 F 1 "Q_PMOS_GDS" H 5450 4450 50  0000 L CNN
 F 2 "TO_SOT_Packages_THT:TO-220-3_Vertical" H 5450 4600 50  0001 C CNN
