File: mk4-v1-board-with-fixes/kicad/hitchco-mk4-mcu.sch (KiCad schematic (older format))
At the start: 1 part

Commit message: Soft push of v2 board modifications
Parts:
- added D?: LED, LEDs:LED_D5.0mm, symbol LED
- added D? (x2): DIODE, symbol DIODE
- added Q?: 2N3904, TO_SOT_Packages_THT:TO-92_Molded_Narrow, symbol 2N3904
- added Q? (x4): Q_PMOS_GDS, TO_SOT_Packages_THT:TO-220-3_Vertical, symbol Q_PMOS_GDS
- added R? (x3): 1KΩ, Resistors_THT:R_Axial_DIN0207_L6.3mm_D2.5mm_P10.16mm_Horizontal, symbol R
- added R?: 560Ω, Resistors_THT:R_Axial_DIN0207_L6.3mm_D2.5mm_P10.16mm_Horizontal, symbol R
- added R? (x5): 10KΩ, Resistors_THT:R_Axial_DIN0207_L6.3mm_D2.5mm_P10.16mm_Horizontal, symbol R
- added R?: 330Ω, Resistors_THT:R_Axial_DIN0207_L6.3mm_D2.5mm_P10.16mm_Horizontal, symbol R
- added U?: CPC1977, symbol CPC1017N
- added U?: CD4013B, symbol CD4013B
Connections:
- net DIRL: now also D?.K, Q?.2 (D)
- net DIRR: now also D?.K, Q?.2 (D)
- net GND: now also Q?.1 (E), R?.1, R?.2, R?.2, R?.2, U?.11 (CLOCK2), U?.4 (RESET1), U?.6 (SET1), U?.7 (VSS), U?.9 (D2)
- net LED1+: now also Q?.3 (S), Q?.3 (S), Q?.3 (S), Q?.3 (S), R?.2, R?.2, R?.2, U?.14 (VDD)
- net PB3_NO: now also R?.1, U?.10 (RESET2)
- net PSU3_GND: now also Q?.2 (D)
- net WIPEL: now also U?.4 (INOUT1)
- net WIPEO: now also R?.2, U?.3 (INOUT2)
- net WIPEO_EN_PIN: now also D?.2 (A), R?.2
- net TACK_SIG_PIN: now reaches SHIELD1.2
- net 3V3: now reaches SHIELD1.3V3
- new net: Q?.2 (B), R?.1, R?.2
- new net: Q?.3 (C), U?.2 (CATH)
- new net: R?.1, U?.1 (ANOD)
- new net: D?.1 (K), R?.1
- new net: R?.1, U?.1 (Q1)
- new net: U?.13 (Q2), U?.3 (CLOCK1)
- new net: U?.2 (~Q1), U?.5 (D1)
- new net: Q?.1 (G), R?.2
- new net FLSHEN: Q?.2 (D)
- new net FLSHIN: D?.A, D?.A
- new net NMOS1_B/DRAIN: Q?.1 (G), R?.1
- new net NMOS1_C/DRAIN: Q?.1 (G), R?.1
- new net NMOS1_D/DRAIN: Q?.1 (G), R?.1
- new net PB3_NC: R?.1, U?.8 (SET2)
- no-connect marks 40 -> 39
