File: mk4-v1-board-with-fixes/kicad/hitchco-mk4.sch (KiCad schematic (older format))
At the start: 22 parts, among them J1 Screw_Terminal_01x10, J10 Conn_02x03_Counter_Clockwise, J12 Conn_02x03_Counter_Clockwise, J13 Conn_02x03_Counter_Clockwise, J15 Conn_02x03_Counter_Clockwise, J16 Conn_02x03_Counter_Clockwise, J18 Conn_02x03_Counter_Clockwise, J19 Conn_02x03_Counter_Clockwise, J2 Screw_Terminal_01x10, J21 Conn_02x03_Counter_Clockwise, J22 Conn_02x03_Counter_Clockwise, J24 Conn_02x03_Counter_Clockwise, J25 Conn_02x03_Counter_Clockwise, J26 Conn_02x03_Counter_Clockwise, J27 Conn_02x03_Counter_Clockwise, J28 Conn_02x03_Counter_Clockwise, J30 Conn_02x03_Counter_Clockwise, J4 Screw_Terminal_01x10, J5 Conn_02x03_Counter_Clockwise, J6 Screw_Terminal_01x10, J7 Conn_02x03_Counter_Clockwise, J8 Conn_02x03_Counter_Clockwise

Commit message: Soft push of v2 board modifications
Changed lines of the file:
@@
 LIBS:valves
 LIBS:freetronics_schematic
+LIBS:cd4013b
 LIBS:hitchco-mk4-cache
 EELAYER 25 0
@@
 $Descr USLedger 11000 17000 portrait
 encoding utf-8
-Sheet 1 47
+Sheet 1 45
 Title "Hitchco MK4"
 Date "2017-10-11"
@@
 P 4100 5100
 F 0 "J10" H 4150 5350 50  0000 C CNN
-F 1 "Conn_02x03_Counter_Clockwise" H 4150 4900 50  0000 C CNN
+F 1 "Conn_02x03_Counter_Clockwise" H 3100 5100 50  0000 C CNN
 F 2 "Socket_Strips:Socket_Strip_Straight_2x03_Pitch2.54mm" H 4100 5100 50  0001 C CNN
 F 3 "" H 4100 5100 50  0001 C CNN
@@
 F108 "HALR" I R 6650 2400 60
 F109 "PB11_LED-" O L 5350 7750 60
+F110 "TACK" I R 6650 4600 60
+F111 "FLSHEN" O R 6650 4850 60
+F112 "FLSHIN" I R 6650 4950 60
+F113 "PB3_NC" I L 5350 5300 60
 $EndSheet
 NoConn ~ 3900 3450
