File: mk4-v2-final/kicad/hitchco-mk4-mcu.sch (KiCad schematic (older format))
At the start: 24 parts

Commit message: got most of the screw terminals planned out in schem
Parts:
- removed Q? (x2): Q_PMOS_GDS, TO_SOT_Packages_THT:TO-220-3_Vertical, symbol Q_PMOS_GDS
- removed R? (x2): 10KΩ, Resistors_THT:R_Axial_DIN0207_L6.3mm_D2.5mm_P10.16mm_Horizontal, symbol R
- added R?: 10KΩ, Resistors_THT:R_Axial_DIN0207_L6.3mm_D2.5mm_P10.16mm_Horizontal, symbol R
Connections:
- net VBAT+ is gone; now on net LED1+: U?.2 (+VIN)
- net VIN(5V) is gone; now on net 5V: SHIELD1.5V, SHIELD1.5V_4, SHIELD1.5V_5
- net GND: now also R?.1
- net LED1_EN_PIN: now also SHIELD1.12
- net RPI_RX: now reaches SHIELD1.14 (TX3)
- net RPI_TX: now reaches SHIELD1.15 (RX3)
- net LDR_SIG_PIN: now reaches SHIELD1.AD14
- net LDR_SIG_PIN: now also R?.2
- no-connect marks 33 -> 29
Other:
- moved on the sheet: SHIELD1

Commit message: added headnight diodes, I don't think software control of them is going to be possible
Parts:
- removed D? (x2): DIODE, symbol DIODE
- added D? (x4): D, symbol D
- gave numbers to parts that had none: 18
Connections:
- net DIRL: now also D?.1 (K)
- net DIRR: now also D?.1 (K)
- net FLSHIN: now also D?.2 (A), D?.2 (A)
- net HLH: now also D?.1 (K)
- net HLL: now also D?.1 (K), D?.2 (A)
- net PKLT: now also D?.2 (A)

Commit message: schematic is done, footprint association and netlist are also done
Parts:
- removed D1: LED, LEDs:LED_D5.0mm, symbol LED
- removed R10: 330Ω, Resistors_THT:R_Axial_DIN0207_L6.3mm_D2.5mm_P10.16mm_Horizontal, symbol R
- removed U2: CPC1977, symbol CPC1017N
- added C16: 0.1uF, C_Rect_L5.08mm_W3.175mm_P2.54mm:C_Rect_L5.08mm_W3.175mm_P2.54mm, symbol C
- added D4, D5: WP7113ID, LEDs:LED_D5.0mm, symbol LED
- added JP1: Jumper, Diodes_THT:D_DO-201AD_P15.24mm_Horizontal, symbol Jumper
- added R30: 10KΩ, Resistors_THT:R_Axial_DIN0204_L3.6mm_D1.6mm_P5.08mm_Horizontal, symbol R
- added R34: 5.1KΩ, Resistors_THT:R_Axial_DIN0204_L3.6mm_D1.6mm_P5.08mm_Horizontal, symbol R
- added R41, R45: 330Ω, Resistors_THT:R_Axial_DIN0204_L3.6mm_D1.6mm_P5.08mm_Horizontal, symbol R
- added U2: LCA715, Housings_DIP:DIP-6_W7.62mm_Socket, symbol LCA715
- D2, D3, D7, D8: renamed from D?; value D -> SB5100E-G; footprint (none) -> Diodes_THT:D_DO-201AD_P15.24mm_Horizontal; digikey-pn (none) -> 641-1421-1-ND; mfg-pn (none) -> SB5100E-G
- Q1: footprint TO_SOT_Packages_THT:TO-92_Molded_Narrow -> TO_SOT_Packages_THT:TO-92_Inline_Wide; digikey-pn (none) -> 2N3904FS-ND; mfg-pn (none) -> 2N3904BU
- Q2: value Q_PMOS_GDS -> NTB5605PT4G; footprint TO_SOT_Packages_THT:TO-220-3_Vertical -> TO_SOT_Packages_SMD:TO-263-3_TabPin2; digikey-pn (none) -> NTB5605PT4GOSCT-ND; mfg-pn (none) -> NTB5605PT4G
- R1, R8, R9: footprint Resistors_THT:R_Axial_DIN0207_L6.3mm_D2.5mm_P10.16mm_Horizontal -> Resistors_THT:R_Axial_DIN0204_L3.6mm_D1.6mm_P5.08mm_Horizontal; digikey-pn (none) -> BC10.0KXCT-ND; mfg-pn (none) -> MBA02040C1002FRP00
- R11, R12, R7: footprint Resistors_THT:R_Axial_DIN0207_L6.3mm_D2.5mm_P10.16mm_Horizontal -> Resistors_THT:R_Axial_DIN0204_L3.6mm_D1.6mm_P5.08mm_Horizontal; digikey-pn (none) -> BC1.00KXCT-ND; mfg-pn (none) -> MBA02040C1001FRP00
- R2, R3, R4, R5: footprint (none) -> Resistors_THT:R_Axial_DIN0204_L3.6mm_D1.6mm_P5.08mm_Horizontal; digikey-pn (none) -> BC1.00KXCT-ND; mfg-pn (none) -> MBA02040C1001FRP00
- R6: footprint Resistors_THT:R_Axial_DIN0207_L6.3mm_D2.5mm_P10.16mm_Horizontal -> Resistors_THT:R_Axial_DIN0204_L3.6mm_D1.6mm_P5.08mm_Horizontal; digikey-pn (none) -> BC3282CT-ND; mfg-pn (none) -> MBA02040C5600FCT00
- U1: digikey-pn (none) -> 811-3084-ND; mfg-pn (none) -> NCS3S1205SC
- U3: footprint (none) -> Housings_DIP:DIP-14_W7.62mm_Socket; digikey-pn (none) -> 296-2033-5-ND; mfg-pn (none) -> CD4013BE
Connections:
- net GND: now also C16.1, R34.2, R41.2, R45.2
- net HORN: now also JP1.1
- net LED1+: now also C16.2
- net PKLT: now also R30.1
- net WIPEL: now also U2.6 (Load)
- net WIPEO: now also U2.4 (Load)
- net at SHIELD1.47 (PL2): now also D4.2 (A)
- net at SHIELD1.48 (PL1): now also D5.2 (A)
- net LITE_SIG_PIN: now reaches SHIELD1.AD15
- net LITE_SIG_PIN: now also R30.2, R34.1
- net at Q1.3 (C): now also U2.2 (-Control)
- net at R6.1: now also U2.1 (+Control)
- net CLK1: now reaches U3.13 (Q2), U3.3 (CLOCK1)
- new net: D4.1 (K), R41.1
- new net: D5.1 (K), R45.1
- new net PB5_LED-: JP1.2
- no-connect marks 29 -> 30
Other:
- note added: "Blinkers & Hazards"
- note added: "Combo Pad Buttons"
- note added: "Headnights\n"
- note added: "Horn\n"
- note added: "LDR Input\n"
- note added: "Other Dash Buttons"
- note added: "Outputs To Car"
- note added: "Raspberry Pi Serial Communication\n"
- note added: "Signals From Car"
- note added: "System Power\n"
- note added: "UI Input Processing"
- note added: "User Input"
- note added: "Wipers\n"
- moved on the sheet: D2, D3, D7, D8, Q1, Q2, R1, R11, R12, R2, R3, R4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

Commit message: all components on the board
Parts:
- Q1: footprint TO_SOT_Packages_THT:TO-92_Inline_Wide -> TO_SOT_Packages_THT:TO-92_Inline_Narrow_Oval
Changed lines of the file:
@@
 F 0 "Q1" H 3300 4375 50  0000 L CNN
 F 1 "2N3904" H 3300 4300 50  0000 L CNN
-F 2 "TO_SOT_Packages_THT:TO-92_Inline_Wide" H 3300 4225 50  0001 L CIN
+F 2 "TO_SOT_Packages_THT:TO-92_Inline_Narrow_Oval" H 3300 4225 50  0001 L CIN
 F 3 "https://www.fairchildsemi.com/datasheets/MM/MMBT3904.pdf" H 3100 4300 50  0001 L CNN
 F 4 "2N3904FS-ND" H 3100 4300 60  0001 C CNN "digikey-pn"
