File: kicad/hitchco-mk4-mcu.sch (KiCad schematic (older format))
At the start: 29 parts, among them Q1 2N3904, Q2 NTB5605PT4G, U1 NCS3S1205SC, U2 LCA715, U3 CD4013B

Commit message: images up
Other:
- note added: "Headlights\n"
- note removed: "Headnights\n"
Changed lines of the file:
@@
 encoding utf-8
 Sheet 2 54
-Title ""
+Title "Hitchco MK4"
 Date "2017-10-11"
-Rev "0.1"
+Rev "1"
 Comp "Hitchcock Management"
 Comment1 ""
@@
 Horn\n
 Text Notes 11450 1050 0    60   ~ 0
-Headnights\n
+Headlights\n
 Text Notes 14350 1050 0    60   ~ 0
 Raspberry Pi Serial Communication\n
