File: kicad/rgbpushbutton.sch (KiCad schematic (older format))
At the start: 1 part

Commit message: images up
Parts:
- R60: value 10K -> 10KΩ
Changed lines of the file:
@@
 encoding utf-8
 Sheet 32 54
-Title ""
+Title "Hitchco MK4"
 Date ""
-Rev ""
-Comp ""
+Rev "1"
+Comp "Hitchcock Management"
 Comment1 ""
 Comment2 ""
@@
 P 5550 4850
 F 0 "R60" V 5630 4850 50  0000 C CNN
-F 1 "10K" V 5550 4850 39  0000 C CNN
+F 1 "10KΩ" V 5550 4850 39  0000 C CNN
 F 2 "Resistors_THT:R_Axial_DIN0204_L3.6mm_D1.6mm_P5.08mm_Horizontal" V 5480 4850 50  0001 C CNN
 F 3 "" H 5550 4850 50  0001 C CNN
